Commit message: modify urdf and parameters to fit so-101 robot

File: src/lekiwi/config/lekiwi.ros2_control.xacro (robot description, xacro)
@@ -17,5 +17,5 @@
         </xacro:unless>
       </hardware>
-      <joint name="Shoulder_Rotation">
+      <joint name="shoulder_pan">
         <command_interface name="position" />
         <state_interface name="position">
@@ -24,5 +24,5 @@
         <!-- <state_interface name="velocity"/> -->
       </joint>
-      <joint name="Shoulder_Pitch">
+      <joint name="shoulder_lift">
         <command_interface name="position" />
         <state_interface name="position">
@@ -31,5 +31,5 @@
         <!-- <state_interface name="velocity"/> -->
       </joint>
-      <joint name="Elbow">
+      <joint name="elbow_flex">
         <command_interface name="position" />
         <state_interface name="position">
@@ -38,5 +38,5 @@
         <!-- <state_interface name="velocity"/> -->
       </joint>
-      <joint name="Wrist_Pitch">
+      <joint name="wrist_flex">
         <command_interface name="position" />
         <state_interface name="position">
@@ -45,5 +45,5 @@
         <!-- <state_interface name="velocity"/> -->
       </joint>
-      <joint name="Wrist_Roll">
+      <joint name="wrist_roll">
         <command_interface name="position" />
         <state_interface name="position">
@@ -52,5 +52,5 @@
         <!-- <state_interface name="velocity"/> -->
       </joint>
-      <joint name="Gripper">
+      <joint name="gripper">
         <command_interface name="position" />
         <state_interface name="position">

File: src/lekiwi/urdf/lekiwi_complete.urdf (robot description, URDF)
Before this commit: robot LeKiwi, 52 links, 51 joints
Links:
- removed link Camera-Model-v3-1
- removed link Fixed_Gripper
- removed link Lower_Arm
- removed link Moving_Jaw
- removed link Moving_Jaw_08d-v1
- removed link Rotation_Pitch_08i-v1
- removed link SO_ARM100_08k_116_Square-v1
- removed link SO_ARM100_08k_Asym_Mirror_Clip-v1
- removed link SO_ARM100_08k_Mirror-v1
- removed link STS3215_03a-v1-1
- removed link STS3215_03a-v1-2
- removed link STS3215_03a-v1-3
- removed link STS3215_03a-v1-4
- removed link STS3215_03a_Wrist_Roll-v1
- removed link Shoulder_Rotation_Pitch
- removed link Upper_Arm
- removed link Wrist-Camera-Mount-v11
- removed link Wrist_Pitch_Roll
- removed link Wrist_Roll_08c-v1
- removed link Wrist_Roll_Pitch_08i-v1
- added link camera, mass 1e-9
- added link gripper_frame_link, mass 1e-9
- added link gripper_link, mass 0.087; collision mesh filename=file://$(find so_100_arm)/urdf/assets/sts3215_03a_v1.stl; collision mesh filename=file://$(find so_100_arm)/urdf/assets/wrist_roll_follower_s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
- added link lower_arm_link, mass 0.104; collision mesh filename=file://$(find so_100_arm)/urdf/assets/motor_holder_so101_wr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; collision mesh filename=file://$(find so_100_arm)/urdf/assets/sts3215_03a_v1.stl
- added link moving_jaw_so101_v1_link, mass 0.012; collision mesh filename=file://$(find so_100_arm)/urdf/assets/moving_jaw_so101_v1.s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; visual mesh filename=file://$(find so_100_arm)/urdf/assets/moving_jaw_so101_v1.s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
- added link shoulder_link, mass 0.100006; collision mesh filename=file://$(find so_100_arm)/urdf/assets/motor_holder_so101_ba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; collision mesh filename=file://$(find so_100_arm)/urdf/assets/rotation_pitch_so101_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
- added link upper_arm_link, mass 0.103; collision mesh filename=file://$(find so_100_arm)/urdf/assets/sts3215_03a_v1.stl; collision mesh filename=file://$(find so_100_arm)/urdf/assets/upper_arm_so101_v1.stl
- added link wrist_link, mass 0.079; collision mesh filename=file://$(find so_100_arm)/urdf/assets/sts3215_03a_no_horn_v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; collision mesh filename=file://$(find so_100_arm)/urdf/assets/wrist_roll_pitch_so10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
Joints:
- removed joint Elbow
- removed joint Gripper
- removed joint Rotation_Pitch_08i-v1_Rigid-46
- removed joint Rotation_Pitch_08i-v1_Rigid-48
- removed joint SO_ARM100_08k_116_Square-v1_Rigid-50
- removed joint SO_ARM100_08k_Mirror-v1_Rigid-52
- removed joint Shoulder_Pitch
- removed joint Shoulder_Rotation
- removed joint Wrist-Camera-Mount-v11_Rigid-71
- removed joint Wrist_Pitch
- removed joint Wrist_Roll
- removed joint Wrist_Roll_08c-v1_Rigid-56
- removed joint Wrist_Roll_08c-v1_Rigid-58
- removed joint Wrist_Roll_Pitch_08i-v1_Rigid-54
- removed joint base_to_shoulder_rotation_pitch
- removed joint elbow_to_lower_arm
- removed joint gripper_to_moving_jaw
- removed joint shoulder_to_upper_arm
- removed joint wrist_roll_to_fixed_gripper
- removed joint wrist_to_wrist_pitch_roll
- added joint camera_frame_joint: type fixed, parent gripper_link, child camera, origin xyz=-0.00 -0.08 -0.00 rpy=-0.445 3.14159 0, axis 0 0 0
- added joint elbow_flex: type revolute, parent upper_arm_link, child lower_arm_link, origin xyz=-0.11257 -0.028 1.73763e-16 rpy=-3.63608e-16 8.74301e-16 1.5708, axis 0 0 1, limit lower=-1.69 upper=1.69 effort=10 velocity=10
- added joint gripper: type revolute, parent gripper_link, child moving_jaw_so101_v1_link, origin xyz=0.0202 0.0188 -0.0234 rpy=1.5708 -5.24284e-08 -1.41553e-15, axis 0 0 1, limit lower=-0.174533 upper=1.74533 effort=10 velocity=10
- added joint gripper_frame_joint: type fixed, parent gripper_link, child gripper_frame_link, origin xyz=-0.0079 -0.000218121 -0.0981274 rpy=0 3.14159 0, axis 0 0 0
- added joint shoulder_lift: type revolute, parent shoulder_link, child upper_arm_link, origin xyz=-0.0303992 -0.0182778 -0.0542 rpy=-1.5708 -1.5708 0, axis 0 0 1, limit lower=-1.74533 upper=1.74533 effort=10 velocity=10
- added joint shoulder_pan: type continuous, parent STS3215_03a-v1, child shoulder_link, origin xyz=-0.010250000000000084 0.03459999999999999 -0.032799999999999996 rpy=1.5707963267948966 -1.5707963267948966 3.94430452610506e-31, axis -3.944304526105059e-31 3.944304526105059e-31 1.0
- added joint wrist_flex: type revolute, parent lower_arm_link, child wrist_link, origin xyz=-0.1349 0.0052 3.62355e-17 rpy=4.02456e-15 8.67362e-16 -1.5708, axis 0 0 1, limit lower=-1.65806 upper=1.65806 effort=10 velocity=10
- added joint wrist_roll: type revolute, parent wrist_link, child gripper_link, origin xyz=5.55112e-17 -0.0611 0.0181 rpy=1.5708 0.0486795 3.14159, axis 0 0 1, limit lower=-2.74385 upper=2.84121 effort=10 velocity=10
