Commit message: change nav2 controller, update urdf

File: src/lekiwi/urdf/lekiwi_complete.urdf (robot description, URDF)
Before this commit: robot LeKiwi, 40 links, 39 joints
Joints:
- joint shoulder_pan: axis -3.944304526105059e-31 3.944304526105059e-31 1.0 -> 0 0 1; limit (none) -> lower=-1.91986 upper=1.91986 effort=10 velocity=10; type continuous -> revolute

Commit message: tuning nav2 params, add new camera

File: src/lekiwi/urdf/lekiwi_complete.urdf (robot description, URDF)
Before this commit: robot LeKiwi, 40 links, 39 joints
Links:
- added link base_camera, mass 1e-9
Joints:
- added joint base_camera_frame_joint: type fixed, parent base_link, child base_camera, origin xyz=-0.00 0.07 0.018 rpy=-1.5708 0 0., axis 0 0 0
